File: BUTTONS.kicad_pcb (KiCad board)
At the start: 2 copper layers, 60 x 30 mm, 15 parts, among them J4 Conn_01x10_Pin, U1 ITR1201SR10AR, U2 ITR1201SR10AR, U3 ITR1201SR10AR, U4 ITR1201SR10AR

Commit message: Add files via upload
Parts:
- LD1: footprint LED_THT:LED_D5.0mm -> LED_SMD:LED_0805_2012Metric_Pad1.15x1.40mm_HandSolder
- moved R5 42.8 mm to (111.9, 123.8)
- moved LD1 36.6 mm to (119.0, 124.0), turned to 180 degrees
Connections:
- net Net-(LD1-A) renamed /LED
- LD1 pad 1: +3.3V -> GNDD
Routing:
- net GNDD: track 205.4 -> 21.9 mm, vias 0 -> 1
- net +3.3V: track 194.0 -> 69.5 mm, vias 0 -> 4
- net /LED: track 6.75 -> 5.25 mm
- net /K4: track 37.1 -> 35.9 mm
- added copper zone on B.Cu, net +3.3V
- added copper zone on F.Cu, net GNDD
Other:
- board text added: "(c) Alex, 2023"
